Commit message: add cr3 robot mock ros2_control launch

File: cr3_moveit/config/cr3_robot.ros2_control.xacro (robot description, xacro)
@@ -1,11 +1,17 @@
 <?xml version="1.0"?>
 <robot xmlns:xacro="http://www.ros.org/wiki/xacro">
-    <xacro:macro name="cr3_robot_ros2_control" params="name initial_positions_file">
-        <xacro:property name="initial_positions" value="${load_yaml(initial_positions_file)['initial_positions']}"/>
+    <xacro:macro name="cr3_robot_ros2_control" params="name initial_positions_file use_mock_hardware:=true robot_ip:=''">
+        <xacro:property name="initial_positions" value="${xacro.load_yaml(initial_positions_file)['initial_positions']}"/>
         <ros2_control name="${name}" type="system">
             <hardware>
-                <!-- By default, set up controllers for simulation. This won't work on real hardware -->
-                <plugin>mock_components/GenericSystem</plugin>
+                <xacro:if value="${use_mock_hardware}">
+                    <plugin>mock_components/GenericSystem</plugin>
+                </xacro:if>
+                <xacro:unless value="${use_mock_hardware}">
+                    <plugin>dobot_hardware_interface/DobotHardwareInterface</plugin>
+                    <param name="robot_ip">${robot_ip}</param>
+                </xacro:unless>
             </hardware>
+            <!-- Joint 1 -->
             <joint name="joint1">
                 <command_interface name="position"/>
@@ -15,4 +21,5 @@
                 <state_interface name="velocity"/>
             </joint>
+            <!-- Joint 2 -->
             <joint name="joint2">
                 <command_interface name="position"/>
@@ -22,4 +29,5 @@
                 <state_interface name="velocity"/>
             </joint>
+            <!-- Joint 3 -->
             <joint name="joint3">
                 <command_interface name="position"/>
@@ -29,4 +37,5 @@
                 <state_interface name="velocity"/>
             </joint>
+            <!-- Joint 4 -->
             <joint name="joint4">
                 <command_interface name="position"/>
@@ -36,4 +45,5 @@
                 <state_interface name="velocity"/>
             </joint>
+            <!-- Joint 5 -->
             <joint name="joint5">
                 <command_interface name="position"/>
@@ -43,4 +53,5 @@
                 <state_interface name="velocity"/>
             </joint>
+            <!-- Joint 6 -->
             <joint name="joint6">
                 <command_interface name="position"/>

File: cr3_moveit/config/cr3_robot.urdf.xacro (robot description, xacro)
@@ -2,8 +2,15 @@
 <robot xmlns:xacro="http://www.ros.org/wiki/xacro" name="cr3_robot">
     <xacro:arg name="initial_positions_file" default="initial_positions.yaml" />
+    <xacro:arg name="use_mock_hardware" default="true" />
+    <xacro:arg name="robot_ip" default="" />
     <!-- Import cr3_robot urdf file -->
     <xacro:include filename="$(find dobot_rviz)/urdf/cr3_robot.urdf" />
     <!-- Import control_xacro -->
     <xacro:include filename="cr3_robot.ros2_control.xacro" />
-    <xacro:cr3_robot_ros2_control name="FakeSystem" initial_positions_file="$(arg initial_positions_file)"/>
+    <xacro:cr3_robot_ros2_control
+        name="dobot_cr3"
+        robot_ip="$(arg robot_ip)"
+        use_mock_hardware="$(arg use_mock_hardware)"
+        initial_positions_file="$(arg initial_positions_file)"
+    />
 </robot>
