Commit message: add nova ros2 control launch, generalize ros2 control launch file

File: nova2_moveit/config/nova2_robot.ros2_control.xacro (robot description, xacro)
@@ -1,10 +1,15 @@
 <?xml version="1.0"?>
 <robot xmlns:xacro="http://www.ros.org/wiki/xacro">
-    <xacro:macro name="nova2_robot_ros2_control" params="name initial_positions_file">
-        <xacro:property name="initial_positions" value="${load_yaml(initial_positions_file)['initial_positions']}"/>
+    <xacro:macro name="nova2_robot_ros2_control" params="name initial_positions_file use_mock_hardware:=true robot_ip:=''">
+        <xacro:property name="initial_positions" value="${xacro.load_yaml(initial_positions_file)['initial_positions']}"/>
         <ros2_control name="${name}" type="system">
             <hardware>
-                <!-- By default, set up controllers for simulation. This won't work on real hardware -->
-                <plugin>mock_components/GenericSystem</plugin>
+                <xacro:if value="${use_mock_hardware}">
+                    <plugin>mock_components/GenericSystem</plugin>
+                </xacro:if>
+                <xacro:unless value="${use_mock_hardware}">
+                    <plugin>dobot_hardware_interface/DobotHardwareInterface</plugin>
+                    <param name="robot_ip">${robot_ip}</param>
+                </xacro:unless>
             </hardware>
             <joint name="joint1">

File: nova2_moveit/config/nova2_robot.urdf.xacro (robot description, xacro)
@@ -2,8 +2,15 @@
 <robot xmlns:xacro="http://www.ros.org/wiki/xacro" name="nova2_robot">
     <xacro:arg name="initial_positions_file" default="initial_positions.yaml" />
+    <xacro:arg name="use_mock_hardware" default="true" />
+    <xacro:arg name="robot_ip" default="" />
     <!-- Import nova2_robot urdf file -->
     <xacro:include filename="$(find dobot_rviz)/urdf/nova2_robot.urdf" />
     <!-- Import control_xacro -->
     <xacro:include filename="nova2_robot.ros2_control.xacro" />
-    <xacro:nova2_robot_ros2_control name="FakeSystem" initial_positions_file="$(arg initial_positions_file)"/>
+    <xacro:nova2_robot_ros2_control
+        name="dobot_nova2"
+        robot_ip="$(arg robot_ip)"
+        use_mock_hardware="$(arg use_mock_hardware)"
+        initial_positions_file="$(arg initial_positions_file)"
+    />
 </robot>
